File: ethoscope_stepper_controller.kicad_pcb (KiCad board)
At the start: 2 copper layers, 74.9 x 74.9 mm, 69 parts, among them P1 PWR_JACK_2.1x5.5_SMD_VERT, T1 TERM_BLK, T2 TERM_BLK, T3 TERM_BLK, T4 TERM_BLK, T5 TERM_BLK, T6 TERM_BLK, T7 TERM_BLK, U1 TMC429, U10 DRV8846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

Commit message: Added autorouted tracks.
Routing:
- net GND: track 0.00 -> 464.4 mm, vias 0 -> 9
- net VAA: track 0.00 -> 145.8 mm, vias 0 -> 6
- net +3V3: track 0.00 -> 145.4 mm, vias 0 -> 4
- net /ENABLE_ALL: track 0.00 -> 140.4 mm, vias 0 -> 7
- net /CS_429_2: track 0.00 -> 81.1 mm
- net /tmc429_0/DIR_1: track 0.00 -> 73.2 mm
- net /tmc429_2/DIR_0: track 0.00 -> 70.9 mm, vias 0 -> 2
- net /tmc429_1/STEP_0: track 0.00 -> 67.7 mm, vias 0 -> 2
- net /tmc429_2/STEP_0: track 0.00 -> 66.7 mm, vias 0 -> 2
- net /MOSI: track 0.00 -> 64.5 mm, vias 0 -> 3
- net /CS_429_1: track 0.00 -> 64.2 mm, vias 0 -> 1
- net /tmc429_0/STEP_1: track 0.00 -> 64.0 mm, vias 0 -> 2
- net /tmc429_1/DIR_0: track 0.00 -> 63.9 mm, vias 0 -> 2
- net /tmc429_1/STEP_2: track 0.00 -> 59.1 mm
- net /tmc429_1/DIR_2: track 0.00 -> 54.2 mm, vias 0 -> 2
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Other:
- board text added: "2.1x5.5 Center + +15-18VDC"

Commit message: Moved traces to pass bug check.
Routing:
- net GND: track 464.4 -> 490.5 mm, vias 9 -> 12
- net (no net): track 0.00 -> 1.27 mm
- added copper zone on B.Cu, net GND
- added copper zone on F.Cu, net GND
Other:
- board text added: "Janelia Modular Device ethoscope_stepper_controller part_number: 2005 08/2018 ver 1.0 3x3"
- board text removed: "Janelia Modular Device ethoscope_stepper_controller part_number: 1000 08/2018 ver 1.0 3x3"
