File: ethoscope_stepper_controller_3x3.kicad_pcb (KiCad board)
At the start: 2 copper layers, 74.9 x 74.9 mm, 71 parts, among them P1 PWR_JACK_2.1x5.5_SMD_VERT, T1 TERM_BLK_HDR_4POS_VERT_0.138IN, T2 TERM_BLK_HDR_4POS_VERT_0.138IN, T3 TERM_BLK_HDR_4POS_VERT_0.138IN, T4 TERM_BLK_HDR_4POS_VERT_0.138IN, T5 TERM_BLK_HDR_4POS_VERT_0.138IN, T6 TERM_BLK_HDR_4POS_VERT_0.138IN, T7 TERM_BLK_HDR_4POS_VERT_0.138IN, U1 TMC429, U10 DRV8846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

Commit message: Progress towards v1.3
Parts:
- TEENSY1: value TEENSY_3.5 -> TEENSY_3.5_MIN
Routing:
- net +3V3: track 453.1 -> 383.0 mm, vias 14 -> 10
- net GND: track 439.6 -> 404.8 mm, vias 0 -> 1
- net /~SLEEP: track 125.2 -> 142.2 mm, vias 8 -> 0
- net /ethoscope_3x3/tmc429_1/stepper_driver_1/BISEN: track 18.3 -> 4.69 mm, vias 0 -> 2
- net /ethoscope_3x3/tmc429_1/stepper_driver_2/BISEN: track 4.69 -> 18.1 mm, vias 2 -> 0
- net /ethoscope_3x3/tmc429_0/stepper_driver_0/BISEN: track 6.89 -> 18.4 mm, vias 2 -> 0
- net /ethoscope_3x3/tmc429_1/STEP_0: track 67.7 -> 57.7 mm
- net /ethoscope_3x3/tmc429_1/DIR_0: track 64.0 -> 56.3 mm
- net /~CS_429_2: track 69.2 -> 76.4 mm
- net /ethoscope_3x3/tmc429_0/stepper_driver_2/A_+: track 9.37 -> 16.4 mm
- net /ethoscope_3x3/tmc429_0/stepper_driver_0/VINT: track 5.16 -> 11.6 mm, vias 2 -> 0
- net /ethoscope_3x3/tmc429_1/stepper_driver_0/VINT: track 5.72 -> 11.7 mm, vias 2 -> 0
- net VAA: track 172.0 -> 177.5 mm, vias 9 -> 8
- net /ethoscope_3x3/tmc429_0/stepper_driver_0/A_+: track 9.53 -> 13.0 mm, vias 1 -> 0
- net /ethoscope_3x3/tmc429_0/DIR_2: track 41.6 -> 38.2 mm
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- removed copper zone on F.Cu, net GND
- removed copper zone on B.Cu, net VAA
Other:
- net class SIGNAL: trace_width 0.2032 -> 0.1524; via_dia 0.4064 -> 0.4572
- rule pad_to_mask_clearance: 0.001 -> 0.1016
- rule solder_mask_min_width: 0.1 -> 0.1016
- rule trace_min: 0.2032 -> 0.1016
- rule via_min_size: 0.4064 -> 0.4572
- board text added: "Janelia Modular Device ethoscope_stepper_controller part_number: 2005 04/2019 ver 1.3 3x3"
- board text removed: "Janelia Modular Device ethoscope_stepper_controller part_number: 2005 02/2019 ver 1.2 3x3"

Commit message: Update date
Other:
- board text added: "Janelia Modular Device ethoscope_stepper_controller part_number: 2005 05/2019 ver 1.3 3x3"
- board text removed: "Janelia Modular Device ethoscope_stepper_controller part_number: 2005 04/2019 ver 1.3 3x3"
Changed lines of the file:
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@@
-(kicad_pcb (version 20190331) (host pcbnew "5.1.0-unknown-2bcf38d~82~ubuntu18.04.1")
+(kicad_pcb (version 20190331) (host pcbnew "6.0.0-unknown-09c9db4~86~ubuntu18.04.1")
   (general
     (thickness 1.6)
@@
     (effects (font (size 1.016 1.016) (thickness 0.1905)))
   )
-  (gr_text "Janelia Modular Device\nethoscope_stepper_controller\npart_number: 2005\n04/2019 ver 1.3 3x3" (at 179.705 118.11) (layer "F.SilkS")
+  (gr_text "Janelia Modular Device\nethoscope_stepper_controller\npart_number: 2005\n05/2019 ver 1.3 3x3" (at 179.705 118.11) (layer "F.SilkS")
     (effects (font (size 0.889 0.889) (thickness 0.22225)))
   )
